File: motorphase.kicad_sch (KiCad schematic)
At the start: 9 parts, among them J4 Motor Connection, Q1 CSD88584Q5DCT

Commit message: more placement
Parts:
- J4: footprint Connector_Wire:SolderWire-0.1sqmm_1x01_D0.4mm_OD1mm -> Connector_Wire:SolderWire-0.75sqmm_1x01_D1.25mm_OD2.3mm
- R13, R15, R2, R3, R4: footprint (none) -> Resistor_SMD:R_0402_1005Metric
Changed lines of the file:
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@@
     (property "Reference" "R2" (id 0) (at 153.67 106.68 90))
     (property "Value" "R_Small_US" (id 1) (at 153.67 109.22 90))
-    (property "Footprint" "" (id 2) (at 153.67 104.14 0)
+    (property "Footprint" "Resistor_SMD:R_0402_1005Metric" (id 2) (at 153.67 104.14 0)
       (effects (font (size 1.27 1.27)) hide)
     )
@@
     (property "Reference" "R15" (id 0) (at 97.79 91.44 90))
     (property "Value" "10R" (id 1) (at 97.79 93.98 90))
-    (property "Footprint" "" (id 2) (at 97.79 96.52 0)
+    (property "Footprint" "Resistor_SMD:R_0402_1005Metric" (id 2) (at 97.79 96.52 0)
       (effects (font (size 1.27 1.27)) hide)
     )
@@
     (property "Reference" "R4" (id 0) (at 171.45 125.73 90))
     (property "Value" "R_Small_US" (id 1) (at 171.45 128.27 90))
-    (property "Footprint" "" (id 2) (at 171.45 123.19 0)
+    (property "Footprint" "Resistor_SMD:R_0402_1005Metric" (id 2) (at 171.45 123.19 0)
       (effects (font (size 1.27 1.27)) hide)
     )
@@
       (effects (font (size 1.27 1.27)) (justify left))
     )
-    (property "Footprint" "Connector_Wire:SolderWire-0.1sqmm_1x01_D0.4mm_OD1mm" (id 2) (at 170.18 85.09 0)
+    (property "Footprint" "Connector_Wire:SolderWire-0.75sqmm_1x01_D1.25mm_OD2.3mm" (id 2) (at 170.18 85.09 0)
       (effects (font (size 1.27 1.27)) hide)
     )
@@
     (property "Reference" "R13" (id 0) (at 97.79 73.66 90))
     (property "Value" "10R" (id 1) (at 97.79 76.2 90))
-    (property "Footprint" "" (id 2) (at 97.79 78.74 0)
+    (property "Footprint" "Resistor_SMD:R_0402_1005Metric" (id 2) (at 97.79 78.74 0)
       (effects (font (size 1.27 1.27)) hide)
     )
@@
     (property "Reference" "R3" (id 0) (at 153.67 118.11 90))
     (property "Value" "R_Small_US" (id 1) (at 153.67 120.65 90))
-    (property "Footprint" "" (id 2) (at 153.67 115.57 0)
+    (property "Footprint" "Resistor_SMD:R_0402_1005Metric" (id 2) (at 153.67 115.57 0)
       (effects (font (size 1.27 1.27)) hide)
     )

Commit message: put everything on, need to choose caps
Parts:
- J4: footprint Connector_Wire:SolderWire-0.75sqmm_1x01_D1.25mm_OD2.3mm -> O32controller:SolderWire-Actual_1x01_D1.7mm_OD_2.5mm
Changed lines of the file:
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@@
       (effects (font (size 1.27 1.27)) (justify left))
     )
-    (property "Footprint" "Connector_Wire:SolderWire-0.75sqmm_1x01_D1.25mm_OD2.3mm" (id 2) (at 170.18 85.09 0)
+    (property "Footprint" "O32controller:SolderWire-Actual_1x01_D1.7mm_OD_2.5mm" (id 2) (at 170.18 85.09 0)
       (effects (font (size 1.27 1.27)) hide)
     )
