File: _autosave-O32controller.kicad_pcb (KiCad board)
At the start: 4 copper layers, 27 x 27 mm, 81 parts, among them J1 SWD, J10 3V3, J11 GND, J12 I2C/RS485_2, J2 BATT+, J3 BATT-, J4 Motor Connection, J5 Motor Connection, J6 Motor Connection, J7 BATT+, J8 BATT-, J9 I2C/RS485_1, Q1 CSD88584Q5DCT, Q2 CSD88584Q5DCT, Q3 CSD88584Q5DCT, SW1 RESET, U1 MA702GQ-P, U2 STSPIN32F0A, U3 THVD1420DRLR

Commit message: ahh my resistor schematic is old:
Parts:
- D1: value SBA0540Q -> SDM2U30CSP; footprint Diode_SMD:D_DFN2L -> O32controller:SDM2U30CSP-7
- D5, D6: value PMEG4010ESB -> SDM2U30CSP
- moved D5 23.8 mm to (42.8, 42.5)
- moved D6 18.7 mm to (39.0, 43.4)
- moved L1 0.21 mm to (39.4, 52.2)
Changed lines of the file:
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@@
   (net 87 "Net-(D4-Pad1)")
   (footprint "O32controller:SDM2U30CSP-7" (layer "F.Cu")
-    (at 21.85 50.8)
+    (at 39.016 43.4)
     (property "Sheetfile" "O32controller.kicad_sch")
     (property "Sheetname" "")
@@
       (effects (font (size 0.321024 0.321024) (thickness 0.15)))
     )
-    (fp_text value "PMEG4010ESB" (at 0 0.869493) (layer "F.Fab")
+    (fp_text value "SDM2U30CSP" (at 0 0.869493) (layer "F.Fab")
       (effects (font (size 0.320531 0.320531) (thickness 0.15)))
     )
@@
   )
   (footprint "O32controller:IND_VLS201612CX-220M-1" (layer "F.Cu")
-    (at 39.3225 52.05 180)
+    (at 39.4 52.25 180)
     (property "Sheetfile" "O32controller.kicad_sch")
     (property "Sheetname" "")
@@
     )
   )
-  (footprint "Diode_SMD:D_DFN2L" (layer "F.Cu")
+  (footprint "O32controller:SDM2U30CSP-7" (layer "F.Cu")
     (at 38.9825 50.475 180)
-    (descr "Diode SMD 0402 (1005 Metric), square (rectangular) end terminal, IPC_7351 nominal, (Body size source: http://www.tortai-tech.com/upload/download/2011102023233369053.pdf), generated with kicad-footprint-generator")
-    (tags "diode")
-    (property "Sheetfile" "O32controller.kicad_sch")
-    (property "Sheetname" "")
-    (attr smd)
-    (fp_text reference "D1" (at 0 -1.17) (layer "F.SilkS")
-      (effects (font (size 1 1) (thickness 0.15)))
-    )
-    (fp_text value "SBA0540Q" (at 0 1.17) (layer "F.Fab")
-      (effects (font (size 1 1) (thickness 0.15)))
-    )
-    (fp_text user "${REFERENCE}" (at 0 0) (layer "F.Fab")
-      (effects (font (size 0.25 0.25) (thickness 0.04)))
-    )
-    (fp_circle (center -1.09 0) (end -1.04 0) (layer "F.SilkS") (width 0.1) (fill none))
-    (fp_line (start -0.93 -0.47) (end 0.93 -0.47) (layer "F.CrtYd") (width 0.05))
-    (fp_line (start 0.93 -0.47) (end 0.93 0.47) (layer "F.CrtYd") (width 0.05))
-    (fp_line (start 0.93 0.47) (end -0.93 0.47) (layer "F.CrtYd") (width 0.05))
-    (fp_line (start -0.93 0.47) (end -0.93 -0.47) (layer "F.CrtYd") (width 0.05))
-    (fp_line (start -0.4 0.25) (end -0.4 -0.25) (layer "F.Fab") (width 0.1))
-    (fp_line (start 0.5 -0.25) (end 0.5 0.25) (layer "F.Fab") (width 0.1))
-    (fp_line (start 0.5 0.25) (end -0.5 0.25) (layer "F.Fab") (width 0.1))
-    (fp_line (start -0.3 0.25) (end -0.3 -0.25) (layer "F.Fab") (width 0.1))
-    (fp_line (start -0.5 -0.25) (end 0.5 -0.25) (layer "F.Fab") (width 0.1))
-    (fp_line (start -0.5 0.25) (end -0.5 -0.25) (layer "F.Fab") (width 0.1))
-    (pad "1" smd roundrect (at -0.34 0 180) (size 0.42 0.6) (layers "F.Cu" "F.Paste" "F.Mask") (roundrect_rratio 0.15)
+    (property "Sheetfile" "O32controller.kicad_sch")
+    (property "Sheetname" "")
+    (attr through_hole)
+    (fp_text reference "D1" (at -0.2 -0.9 180) (layer "F.SilkS")
+      (effects (font (size 0.321024 0.321024) (thickness 0.15)))
+    )
+    (fp_text value "SDM2U30CSP" (at -0.2 0.869493 180) (layer "F.Fab")
+      (effects (font (size 0.320531 0.320531) (thickness 0.15)))
+    )
+    (fp_rect (start -1.067 -0.545) (end 1.035 0.545) (layer "F.CrtYd") (width 0.05) (fill none))
+    (fp_rect (start 0.7778 0.4) (end -0.8222 -0.4) (layer "F.Fab") (width 0.05) (fill none))
+    (pad "1" smd rect (at -0.6745 0 180) (size 0.385 0.69) (layers "F.Cu" "F.Paste" "F.Mask")
       (net 68 "/SW_3.3") (pinfunction "K") (pintype "passive"))
-    (pad "2" smd roundrect (at 0.34 0 180) (size 0.42 0.6) (layers "F.Cu" "F.Paste" "F.Mask") (roundrect_rratio 0.15)
+    (pad "2" smd rect (at 0.3175 0 180) (size 1.035 0.69) (layers "F.Cu" "F.Paste" "F.Mask")
       (net 24 "GND") (pinfunction "A") (pintype "passive"))
-    (model "${KICAD6_3DMODEL_DIR}/Diode_SMD.3dshapes/D_0402_1005Metric.wrl"
+    (model "${KIPRJMOD}/O32controller.pretty/DIODE_SDM2U30CSP-7_DIO.step"
       (offset (xyz 0 0 0))
       (scale (xyz 1 1 1))
@@
   )
   (footprint "O32controller:SDM2U30CSP-7" (layer "F.Cu")
-    (at 19.666 48.05)
+    (at 42.8 42.55)
     (property "Sheetfile" "O32controller.kicad_sch")
     (property "Sheetname" "")
@@
       (effects (font (size 0.321024 0.321024) (thickness 0.15)))
     )
-    (fp_text value "PMEG4010ESB" (at 0 0.869493) (layer "F.Fab")
+    (fp_text value "SDM2U30CSP" (at 0 0.869493) (layer "F.Fab")
       (effects (font (size 0.320531 0.320531) (thickness 0.15)))
     )
