File: _autosave-O32controller.kicad_sch (KiCad schematic)
At the start: 42 parts, among them J1 SWD, J10 3V3, J11 GND, J12 I2C/RS485_2, J2 BATT+, J3 BATT-, J7 BATT+, J8 BATT-, J9 I2C/RS485_1, SW1 RESET, U1 MA702GQ-P, U2 STSPIN32F0A, U3 THVD1420DRLR

Commit message: choose led, tvs, start on silkscreen
Parts:
- J10, J11: now left out of the parts list
Changed lines of the file:
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@@
   )
   (symbol (lib_id "Connector_Generic:Conn_01x01") (at 261.62 148.59 0) (unit 1)
-    (in_bom yes) (on_board yes) (fields_autoplaced)
+    (in_bom no) (on_board yes) (fields_autoplaced)
     (property "Reference" "J10" (id 0) (at 264.16 147.3199 0)
       (effects (font (size 1.27 1.27)) (justify left))
@@
   )
   (symbol (lib_id "Connector_Generic:Conn_01x01") (at 261.62 153.67 0) (unit 1)
-    (in_bom yes) (on_board yes) (fields_autoplaced)
+    (in_bom no) (on_board yes) (fields_autoplaced)
     (property "Reference" "J11" (id 0) (at 264.16 152.3999 0)
       (effects (font (size 1.27 1.27)) (justify left))
