File: O12encoder/O12encoder.kicad_sch (KiCad schematic)
At the start: 17 parts, among them J1 Conn_01x06_Pin, J2 Conn_01x06_Pin, J4 Conn_01x06_Pin, J5 JST_SM02B-SRSS-TB(LF)(SN), J6 Conn_01x06_Pin, J7 Conn_01x06_Pin, J8 Conn_01x06_Pin, U1 MA702GQ-P, U2 STM32L011F4Ux, U3 THVD1420DRLR

Commit message: update readme pic
Parts:
- C1: MPN GCM155C71A105KE38D -> CL05A105KA5NQNC; Vendor# C126521 -> C52923
- C2, C3: MPN (none) -> CL05A105KA5NQNC; Vendor (none) -> LCSC; Vendor# (none) -> C52923
- J5: MP SM02B-SRSS-TB_LF__SN_ -> (none); MPN (none) -> SM02B-SRSS-TB(LF)(SN); Vendor (none) -> LCSC; Vendor# (none) -> C160402
- U1: Vendor (none) -> MPS
- U2: MPN STM32L011F4U3TR -> STM32L011F4U6TR; Vendor Digikey -> LCSC; Vendor# (none) -> C329283
- U3: Vendor (none) -> Digikey; Vendor# (none) -> 296-THVD1420DRLRCT-ND
Changed lines of the file:
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@@
+      (effects (font (size 1.27 1.27)) hide)
+    )
+    (property "MPN" "CL05A105KA5NQNC" (at 118.11 39.37 0)
+      (effects (font (size 1.27 1.27)) hide)
+    )
+    (property "Vendor" "LCSC" (at 118.11 39.37 0)
+      (effects (font (size 1.27 1.27)) hide)
+    )
+    (property "Vendor#" "C52923" (at 118.11 39.37 0)
       (effects (font (size 1.27 1.27)) hide)
     )
@@
       (effects (font (size 1.27 1.27)) hide)
     )
-    (property "MP" "SM02B-SRSS-TB_LF__SN_" (at 220.98 77.47 0)
+    (property "MP" "" (at 220.98 77.47 0)
       (effects (font (size 1.27 1.27)) (justify bottom) hide)
+    )
+    (property "MPN" "SM02B-SRSS-TB(LF)(SN)" (at 229.87 59.69 0)
+      (effects (font (size 1.27 1.27)) hide)
+    )
+    (property "Vendor" "LCSC" (at 229.87 59.69 0)
+      (effects (font (size 1.27 1.27)) hide)
+    )
+    (property "Vendor#" "C160402" (at 229.87 59.69 0)
+      (effects (font (size 1.27 1.27)) hide)
     )
     (pin "1")
@@
     )
     (property "MPN" "THVD1420DRLR" (at 234.95 36.83 0)
+      (effects (font (size 1.27 1.27)) hide)
+    )
+    (property "Vendor" "Digikey" (at 234.95 36.83 0)
+      (effects (font (size 1.27 1.27)) hide)
+    )
+    (property "Vendor#" "296-THVD1420DRLRCT-ND" (at 234.95 36.83 0)
       (effects (font (size 1.27 1.27)) hide)
     )
@@
       (effects (font (size 1.27 1.27)) hide)
     )
-    (property "MPN" "STM32L011F4U3TR" (at 138.43 64.77 0)
-      (effects (font (size 1.27 1.27)) hide)
-    )
-    (property "Vendor" "Digikey" (at 138.43 64.77 0)
+    (property "MPN" "STM32L011F4U6TR" (at 138.43 64.77 0)
+      (effects (font (size 1.27 1.27)) hide)
+    )
+    (property "Vendor" "LCSC" (at 138.43 64.77 0)
+      (effects (font (size 1.27 1.27)) hide)
+    )
+    (property "Vendor#" "C329283" (at 138.43 64.77 0)
       (effects (font (size 1.27 1.27)) hide)
     )
@@
       (effects (font (size 1.27 1.27)) hide)
     )
+    (property "MPN" "CL05A105KA5NQNC" (at 152.4 39.37 0)
+      (effects (font (size 1.27 1.27)) hide)
+    )
+    (property "Vendor" "LCSC" (at 152.4 39.37 0)
+      (effects (font (size 1.27 1.27)) hide)
+    )
+    (property "Vendor#" "C52923" (at 152.4 39.37 0)
+      (effects (font (size 1.27 1.27)) hide)
+    )
     (pin "1")
     (pin "2")
@@
       (effects (font (size 1.27 1.27)) hide)
     )
-    (property "Vendor#" "C126521" (at 115.57 115.57 0)
-      (effects (font (size 1.27 1.27)) hide)
-    )
-    (property "MPN" "GCM155C71A105KE38D" (at 115.57 115.57 0)
+    (property "Vendor#" "C52923" (at 115.57 115.57 0)
+      (effects (font (size 1.27 1.27)) hide)
+    )
+    (property "MPN" "CL05A105KA5NQNC" (at 115.57 115.57 0)
       (effects (font (size 1.27 1.27)) hide)
     )
@@
       (effects (font (size 1.524 1.524)))
     )
-    (pin "1")
+    (property "Vendor" "MPS" (at 146.05 143.51 0)
+      (effects (font (size 1.27 1.27)) hide)
+    )
+    (pin "1")
