File: v3/motorphase.kicad_sch (KiCad schematic)
At the start: 15 parts, among them J4 Motor Connection, Q1 CSD88584Q5DCT

Commit message: external spi, update bus sns res, routing
Other:
- company: (none) -> Christopher Xu
Changed lines of the file:
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@@
     (date "2023-12-26")
     (rev "3")
+    (company "Christopher Xu")
   )
   (junction (at 128.27 104.14) (diameter 0) (color 0 0 0 0)

Commit message: bus caps, finished routing?
Parts:
- renumbered C18 to C14, J4 to J10, R13 to R11, R23 to R12, R15 to R13, R30 to R14, R2 to R15, R31 to R16, R3 to R17, R1 to R18, R4 to R19

Commit message: export for PCBway
Parts:
- C12: MP CL05B103KB5NNNC -> (none); MPN (none) -> CL05B103KB5NNNC; Vendor (none) -> LCSC; Vendor# (none) -> C15195
- C13: MP GRM155R72A472KA01D -> (none); MPN (none) -> GRM155R72A472KA01D; Vendor (none) -> LCSC; Vendor# (none) -> C415704
- C14: MP CC0402MRX7R9BB102 -> (none); MPN (none) -> CC0402MRX7R9BB102; Vendor (none) -> LCSC; Vendor# (none) -> C527029
- Q1: value CSD88584Q5DCT -> CSD88584Q5DC; MP CSD88584Q5DCT -> (none); MPN (none) -> CSD88584Q5DC; Vendor (none) -> Digikey; Vendor# (none) -> 296-48904-1-ND
- R11, R13: MP RCS040210R0FKED -> (none); MPN (none) -> SR0402FR-7T10RL; Vendor (none) -> LCSC; Vendor# (none) -> C854481
- R12: MP SG73P1EWTTP2R20F -> (none); MPN (none) -> CRCW04022R20JNEDHP; Vendor (none) -> LCSC; Vendor# (none) -> C2079158
- R14, R16: MP RC0402FR-0727K4L -> (none); MPN (none) -> RC0402FR-0727K4L; Vendor (none) -> LCSC; Vendor# (none) -> C273730
- R15, R17: MP RC0402FR-071K78L -> (none); MPN (none) -> RC0402FR-071K78L; Vendor (none) -> LCSC; Vendor# (none) -> C185450
- R18: value WSLF25122L000FEB 0.002R -> PU2512FKMP50R002L; MP WSLF25122L000FEB 0.002R -> (none); MPN (none) -> PU2512FKMP50R002L; Vendor (none) -> LCSC; Vendor# (none) -> C2090861
- R19: MP RC0402FR-0713K7L -> (none); MPN (none) -> RC0402FR-0713K7L; Vendor (none) -> LCSC; Vendor# (none) -> C274888
Other:
- note added: "1/5W 0402"
- note removed: "1/4W 0402"
Changed lines of the file:
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@@
     (effects (font (size 1.27 1.27)) (justify left bottom))
   )
-  (text "1/4W 0402\n" (at 154.94 80.01 0)
+  (text "1/5W 0402\n" (at 154.94 80.01 0)
     (effects (font (size 1.27 1.27)) (justify left bottom))
   )
@@
       (effects (font (size 1.27 1.27)) hide)
     )
-    (property "MP" "RC0402FR-071K78L " (at 146.05 104.14 0)
+    (property "Vendor" "LCSC" (at 146.05 104.14 0)
+      (effects (font (size 1.27 1.27)) hide)
+    )
+    (property "Vendor#" "C185450" (at 146.05 104.14 0)
+      (effects (font (size 1.27 1.27)) hide)
+    )
+    (property "MPN" "RC0402FR-071K78L " (at 146.05 104.14 0)
       (effects (font (size 1.27 1.27)) hide)
     )
@@
       (effects (font (size 1.27 1.27)) hide)
     )
-    (property "MP" "RCS040210R0FKED " (at 97.79 80.01 0)
+    (property "Vendor" "LCSC" (at 97.79 80.01 0)
+      (effects (font (size 1.27 1.27)) hide)
+    )
+    (property "Vendor#" "C854481" (at 97.79 80.01 0)
+      (effects (font (size 1.27 1.27)) hide)
+    )
+    (property "MPN" "SR0402FR-7T10RL" (at 97.79 80.01 0)
       (effects (font (size 1.27 1.27)) hide)
     )
@@
       (effects (font (size 1.27 1.27)) hide)
     )
-    (property "MP" "SG73P1EWTTP2R20F " (at 146.05 78.74 0)
+    (property "Vendor" "LCSC" (at 146.05 78.74 0)
+      (effects (font (size 1.27 1.27)) hide)
+    )
+    (property "Vendor#" "C2079158" (at 146.05 78.74 0)
+      (effects (font (size 1.27 1.27)) hide)
+    )
+    (property "MPN" "CRCW04022R20JNEDHP" (at 146.05 78.74 0)
       (effects (font (size 1.27 1.27)) hide)
     )
@@
       (effects (font (size 1.27 1.27)) hide)
     )
+    (property "Vendor" "" (at 133.35 130.81 0)
+      (effects (font (size 1.27 1.27)) hide)
+    )
+    (property "Vendor#" "" (at 133.35 130.81 0)
+      (effects (font (size 1.27 1.27)) hide)
+    )
+    (property "MPN" "" (at 133.35 130.81 0)
+      (effects (font (size 1.27 1.27)) hide)
+    )
     (pin "1")
     (pin "2")
@@
       (effects (font (size 1.27 1.27)) hide)
     )
-    (property "MP" "GRM155R72A472KA01D" (at 146.05 72.39 0)
+    (property "Vendor" "LCSC" (at 146.05 72.39 0)
+      (effects (font (size 1.27 1.27)) hide)
+    )
+    (property "Vendor#" "C415704" (at 146.05 72.39 0)
+      (effects (font (size 1.27 1.27)) hide)
+    )
+    (property "MPN" "GRM155R72A472KA01D" (at 146.05 72.39 0)
       (effects (font (size 1.27 1.27)) hide)
     )
@@
       (effects (font (size 1.27 1.27)) hide)
     )
-    (property "MP" "CL05B103KB5NNNC" (at 71.12 69.85 0)
+    (property "Vendor" "LCSC" (at 71.12 69.85 0)
+      (effects (font (size 1.27 1.27)) hide)
+    )
+    (property "Vendor#" "C15195" (at 71.12 69.85 0)
+      (effects (font (size 1.27 1.27)) hide)
+    )
+    (property "MPN" "CL05B103KB5NNNC" (at 71.12 69.85 0)
       (effects (font (size 1.27 1.27)) hide)
     )
@@
       (effects (font (size 1.27 1.27)) hide)
     )
-    (property "MP" "RC0402FR-0727K4L " (at 160.02 101.6 0)
+    (property "Vendor" "LCSC" (at 160.02 101.6 0)
+      (effects (font (size 1.27 1.27)) hide)
+    )
+    (property "Vendor#" "C273730" (at 160.02 101.6 0)
+      (effects (font (size 1.27 1.27)) hide)
+    )
+    (property "MPN" "RC0402FR-0727K4L " (at 160.02 101.6 0)
       (effects (font (size 1.27 1.27)) hide)
     )
@@
       (effects (font (size 1.27 1.27)) hide)
     )
-    (property "MP" "RC0402FR-0727K4L " (at 160.02 106.68 0)
+    (property "Vendor" "LCSC" (at 160.02 106.68 0)
+      (effects (font (size 1.27 1.27)) hide)
+    )
+    (property "Vendor#" "C273730" (at 160.02 106.68 0)
+      (effects (font (size 1.27 1.27)) hide)
+    )
+    (property "MPN" "RC0402FR-0727K4L " (at 160.02 106.68 0)
       (effects (font (size 1.27 1.27)) hide)
     )
@@
       (effects (font (size 1.27 1.27)) hide)
     )
-    (property "MP" "RC0402FR-0713K7L " (at 181.61 123.19 0)
+    (property "Vendor" "LCSC" (at 181.61 123.19 0)
+      (effects (font (size 1.27 1.27)) hide)
+    )
+    (property "Vendor#" "C274888" (at 181.61 123.19 0)
+      (effects (font (size 1.27 1.27)) hide)
+    )
+    (property "MPN" "RC0402FR-0713K7L " (at 181.61 123.19 0)
       (effects (font (size 1.27 1.27)) hide)
     )
@@
       (effects (font (size 1.27 1.27)) hide)
     )
+    (property "Vendor" "" (at 170.18 67.31 0)
+      (effects (font (size 1.27 1.27)) hide)
+    )
+    (property "Vendor#" "" (at 170.18 67.31 0)
+      (effects (font (size 1.27 1.27)) hide)
+    )
+    (property "MPN" "" (at 170.18 67.31 0)
+      (effects (font (size 1.27 1.27)) hide)
+    )
     (pin "1")
     (instances
@@
       (effects (font (size 1.27 1.27)) hide)
     )
-    (property "MP" "CC0402MRX7R9BB102" (at 181.61 134.62 0)
+    (property "Vendor" "LCSC" (at 181.61 134.62 0)
+      (effects (font (size 1.27 1.27)) hide)
+    )
+    (property "Vendor#" "C527029" (at 181.61 134.62 0)
+      (effects (font (size 1.27 1.27)) hide)
+    )
+    (property "MPN" "CC0402MRX7R9BB102" (at 181.61 134.62 0)
       (effects (font (size 1.27 1.27)) hide)
     )
@@
       (effects (font (size 1.524 1.524)) (justify left))
     )
-    (property "Value" "CSD88584Q5DCT" (at 130.4151 59.69 0)
+    (property "Value" "CSD88584Q5DC" (at 130.4151 59.69 0)
       (effects (font (size 1.524 1.524)) (justify left))
     )
@@
       (effects (font (size 1.524 1.524)) (justify left) hide)
     )
-    (property "MP" "CSD88584Q5DCT" (at 128.27 71.12 0)
+    (property "Vendor" "Digikey" (at 128.27 71.12 0)
+      (effects (font (size 1.27 1.27)) hide)
+    )
+    (property "Vendor#" "296-48904-1-ND" (at 128.27 71.12 0)
+      (effects (font (size 1.27 1.27)) hide)
+    )
+    (property "MPN" "CSD88584Q5DC" (at 128.27 71.12 0)
       (effects (font (size 1.27 1.27)) hide)
     )
@@
       (effects (font (size 1.27 1.27)) (justify left))
     )
-    (property "Value" "WSLF25122L000FEB 0.002R" (at 124.46 116.8401 90)
+    (property "Value" "PU2512FKMP50R002L" (at 124.46 116.8401 90)
       (effects (font (size 1.27 1.27)) (justify left))
     )
@@
       (effects (font (size 1.27 1.27)) (justify bottom) hide)
     )
-    (property "Datasheet" "https://www.vishay.com/docs/30193/wslf.pdf" (at 128.27 118.11 0)
-      (effects (font (size 1.27 1.27)) hide)
-    )
-    (property "MP" "WSLF25122L000FEB 0.002R" (at 128.27 118.11 0)
+    (property "Datasheet" "https://datasheet.lcsc.com/lcsc/2304140030_YAGEO-PU2512FKMP50R002L_C2090861.pdf" (at 128.27 118.11 0)
+      (effects (font (size 1.27 1.27)) hide)
+    )
+    (property "Vendor" "LCSC" (at 128.27 118.11 0)
+      (effects (font (size 1.27 1.27)) hide)
+    )
+    (property "Vendor#" "C2090861" (at 128.27 118.11 0)
+      (effects (font (size 1.27 1.27)) hide)
+    )
+    (property "MPN" "PU2512FKMP50R002L" (at 128.27 118.11 0)
       (effects (font (size 1.27 1.27)) hide)
     )
@@
       (effects (font (size 1.27 1.27)) hide)
     )
-    (property "MP" "RCS040210R0FKED " (at 97.79 62.23 0)
+    (property "Vendor" "LCSC" (at 97.79 62.23 0)
+      (effects (font (size 1.27 1.27)) hide)
+    )
+    (property "Vendor#" "C854481" (at 97.79 62.23 0)
+      (effects (font (size 1.27 1.27)) hide)
+    )
+    (property "MPN" "SR0402FR-7T10RL" (at 97.79 62.23 0)
       (effects (font (size 1.27 1.27)) hide)
     )
@@
       (effects (font (size 1.27 1.27)) hide)
     )
-    (property "MP" "RC0402FR-071K78L " (at 146.05 115.57 0)
-      (effects (font (size 1.27 1.27)) hide)
-    )
+    (property "Vendor" "LCSC" (at 146.05 115.57 0)
+      (effects (font (size 1.27 1.27)) hide)
+    )
+    (property "Vendor#" "C185450" (at 146.05 115.57 0)
+      (effects (font (size 1.27 1.27)) hide)
+    )
+    (property "MPN" "RC0402FR-071K78L " (at 146.05 115.57 0)
+      (effects (font (size 1.27 1.27)) hide)
+    )

Commit message: use MA732 instead of 702, SMF15A
Parts:
- C12: LCSC (none) -> C15195
- C13: LCSC (none) -> C415704
- C14: LCSC (none) -> C527029
- R11, R13: LCSC (none) -> C854481
- R12: LCSC (none) -> C2079158
- R14, R16: LCSC (none) -> C273730
- R15, R17: LCSC (none) -> C185450
- R18: LCSC (none) -> C2090861
- R19: LCSC (none) -> C274888
Changed lines of the file:
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@@
+      (effects (font (size 1.27 1.27)) hide)
+    )
+    (property "LCSC" "C185450" (at 146.05 104.14 0)
       (effects (font (size 1.27 1.27)) hide)
     )
@@
     )
     (property "MPN" "SR0402FR-7T10RL" (at 97.79 80.01 0)
+      (effects (font (size 1.27 1.27)) hide)
+    )
+    (property "LCSC" "C854481" (at 97.79 80.01 0)
       (effects (font (size 1.27 1.27)) hide)
     )
@@
       (effects (font (size 1.27 1.27)) hide)
     )
+    (property "LCSC" "C2079158" (at 146.05 78.74 0)
+      (effects (font (size 1.27 1.27)) hide)
+    )
     (pin "1")
     (pin "2")
@@
       (effects (font (size 1.27 1.27)) hide)
     )
+    (property "LCSC" "" (at 133.35 130.81 0)
+      (effects (font (size 1.27 1.27)) hide)
+    )
     (pin "1")
     (pin "2")
@@
     )
     (property "MPN" "GRM155R72A472KA01D" (at 146.05 72.39 0)
+      (effects (font (size 1.27 1.27)) hide)
+    )
+    (property "LCSC" "C415704" (at 146.05 72.39 0)
       (effects (font (size 1.27 1.27)) hide)
     )
@@
       (effects (font (size 1.27 1.27)) hide)
     )
+    (property "LCSC" "C15195" (at 71.12 69.85 0)
+      (effects (font (size 1.27 1.27)) hide)
+    )
     (pin "1")
     (pin "2")
@@
       (effects (font (size 1.27 1.27)) hide)
     )
+    (property "LCSC" "C273730" (at 160.02 101.6 0)
+      (effects (font (size 1.27 1.27)) hide)
+    )
     (pin "1")
     (pin "2")
@@
       (effects (font (size 1.27 1.27)) hide)
     )
+    (property "LCSC" "C273730" (at 160.02 106.68 0)
+      (effects (font (size 1.27 1.27)) hide)
+    )
     (pin "1")
     (pin "2")
@@
     )
     (property "MPN" "RC0402FR-0713K7L " (at 181.61 123.19 0)
+      (effects (font (size 1.27 1.27)) hide)
+    )
+    (property "LCSC" "C274888" (at 181.61 123.19 0)
       (effects (font (size 1.27 1.27)) hide)
     )
@@
       (effects (font (size 1.27 1.27)) hide)
     )
+    (property "LCSC" "" (at 170.18 67.31 0)
+      (effects (font (size 1.27 1.27)) hide)
+    )
     (pin "1")
     (instances
@@
     )
     (property "MPN" "CC0402MRX7R9BB102" (at 181.61 134.62 0)
+      (effects (font (size 1.27 1.27)) hide)
+    )
+    (property "LCSC" "C527029" (at 181.61 134.62 0)
       (effects (font (size 1.27 1.27)) hide)
     )
@@
     )
     (property "MPN" "CSD88584Q5DC" (at 128.27 71.12 0)
+      (effects (font (size 1.27 1.27)) hide)
+    )
+    (property "LCSC" "" (at 128.27 71.12 0)
       (effects (font (size 1.27 1.27)) hide)
     )
@@
       (effects (font (size 1.27 1.27)) hide)
     )
+    (property "LCSC" "C2090861" (at 128.27 118.11 0)
+      (effects (font (size 1.27 1.27)) hide)
+    )
     (pin "1")
     (pin "2")
@@
       (effects (font (size 1.27 1.27)) hide)
     )
+    (property "LCSC" "C854481" (at 97.79 62.23 0)
+      (effects (font (size 1.27 1.27)) hide)
+    )
     (pin "1")
     (pin "2")
@@
       (effects (font (size 1.27 1.27)) hide)
     )
+    (property "LCSC" "C185450" (at 146.05 115.57 0)
+      (effects (font (size 1.27 1.27)) hide)
+    )

Commit message: finalize BOM for v3.1, shared w Axlab
Parts:
- C12: Type (none) -> Basic
- C13: LCSC C415704 -> C1538; MPN GRM155R72A472KA01D -> 0402B472K500NT; Type (none) -> Basic; Vendor# C415704 -> C1538
- C14: LCSC C527029 -> C1523; MPN CC0402MRX7R9BB102 -> 0402B102K500NT; Type (none) -> Basic; Vendor# C527029 -> C1523
- Q1: Type (none) -> Global; Vendor Digikey -> TI; Vendor# 296-48904-1-ND -> CSD88584Q5DC
- R11, R13, R14, R16, R18, R19: Type (none) -> Extended
- R12: LCSC C2079158 -> C131536; MPN CRCW04022R20JNEDHP -> RK73B1ETTP2R2J; Type (none) -> Extended; Vendor# C2079158 -> C131536
- R15, R17: LCSC C185450 -> C284379; MPN RC0402FR-071K78L -> ARG02FTC1781; Type (none) -> Extended; Vendor# C185450 -> C284379
Changed lines of the file:
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@@
       (effects (font (size 1.27 1.27)) hide)
     )
-    (property "Vendor#" "C185450" (at 146.05 104.14 0)
-      (effects (font (size 1.27 1.27)) hide)
-    )
-    (property "MPN" "RC0402FR-071K78L " (at 146.05 104.14 0)
-      (effects (font (size 1.27 1.27)) hide)
-    )
-    (property "LCSC" "C185450" (at 146.05 104.14 0)
+    (property "Vendor#" "C284379" (at 146.05 104.14 0)
+      (effects (font (size 1.27 1.27)) hide)
+    )
+    (property "MPN" "ARG02FTC1781" (at 146.05 104.14 0)
+      (effects (font (size 1.27 1.27)) hide)
+    )
+    (property "LCSC" "C284379" (at 146.05 104.14 0)
+      (effects (font (size 1.27 1.27)) hide)
+    )
+    (property "Type" "Extended" (at 146.05 104.14 0)
       (effects (font (size 1.27 1.27)) hide)
     )
@@
     )
     (property "LCSC" "C854481" (at 97.79 80.01 0)
+      (effects (font (size 1.27 1.27)) hide)
+    )
+    (property "Type" "Extended" (at 97.79 80.01 0)
       (effects (font (size 1.27 1.27)) hide)
     )
@@
       (effects (font (size 1.27 1.27)) hide)
     )
-    (property "Vendor#" "C2079158" (at 146.05 78.74 0)
-      (effects (font (size 1.27 1.27)) hide)
-    )
-    (property "MPN" "CRCW04022R20JNEDHP" (at 146.05 78.74 0)
-      (effects (font (size 1.27 1.27)) hide)
-    )
-    (property "LCSC" "C2079158" (at 146.05 78.74 0)
+    (property "Vendor#" "C131536" (at 146.05 78.74 0)
+      (effects (font (size 1.27 1.27)) hide)
+    )
+    (property "MPN" "RK73B1ETTP2R2J" (at 146.05 78.74 0)
+      (effects (font (size 1.27 1.27)) hide)
+    )
+    (property "LCSC" "C131536" (at 146.05 78.74 0)
+      (effects (font (size 1.27 1.27)) hide)
+    )
+    (property "Type" "Extended" (at 146.05 78.74 0)
       (effects (font (size 1.27 1.27)) hide)
     )
@@
       (effects (font (size 1.27 1.27)) hide)
     )
+    (property "Type" "" (at 133.35 130.81 0)
+      (effects (font (size 1.27 1.27)) hide)
+    )
     (pin "1")
     (pin "2")
@@
       (effects (font (size 1.27 1.27)) hide)
     )
-    (property "Vendor#" "C415704" (at 146.05 72.39 0)
-      (effects (font (size 1.27 1.27)) hide)
-    )
-    (property "MPN" "GRM155R72A472KA01D" (at 146.05 72.39 0)
-      (effects (font (size 1.27 1.27)) hide)
-    )
-    (property "LCSC" "C415704" (at 146.05 72.39 0)
+    (property "Vendor#" "C1538" (at 146.05 72.39 0)
+      (effects (font (size 1.27 1.27)) hide)
+    )
+    (property "MPN" "0402B472K500NT" (at 146.05 72.39 0)
+      (effects (font (size 1.27 1.27)) hide)
+    )
+    (property "LCSC" "C1538" (at 146.05 72.39 0)
+      (effects (font (size 1.27 1.27)) hide)
+    )
+    (property "Type" "Basic" (at 146.05 72.39 0)
       (effects (font (size 1.27 1.27)) hide)
     )
@@
       (effects (font (size 1.27 1.27)) hide)
     )
+    (property "Type" "Basic" (at 71.12 69.85 0)
+      (effects (font (size 1.27 1.27)) hide)
+    )
     (pin "1")
     (pin "2")
@@
       (effects (font (size 1.27 1.27)) hide)
     )
+    (property "Type" "Extended" (at 160.02 101.6 0)
+      (effects (font (size 1.27 1.27)) hide)
+    )
     (pin "1")
     (pin "2")
@@
       (effects (font (size 1.27 1.27)) hide)
     )
+    (property "Type" "Extended" (at 160.02 106.68 0)
+      (effects (font (size 1.27 1.27)) hide)
+    )
     (pin "1")
     (pin "2")
@@
     )
     (property "LCSC" "C274888" (at 181.61 123.19 0)
+      (effects (font (size 1.27 1.27)) hide)
+    )
+    (property "Type" "Extended" (at 181.61 123.19 0)
       (effects (font (size 1.27 1.27)) hide)
     )
@@
       (effects (font (size 1.27 1.27)) hide)
     )
+    (property "Type" "" (at 170.18 67.31 0)
+      (effects (font (size 1.27 1.27)) hide)
+    )
     (pin "1")
     (instances
@@
       (effects (font (size 1.27 1.27)) hide)
     )
-    (property "Vendor#" "C527029" (at 181.61 134.62 0)
-      (effects (font (size 1.27 1.27)) hide)
-    )
-    (property "MPN" "CC0402MRX7R9BB102" (at 181.61 134.62 0)
-      (effects (font (size 1.27 1.27)) hide)
-    )
-    (property "LCSC" "C527029" (at 181.61 134.62 0)
+    (property "Vendor#" "C1523" (at 181.61 134.62 0)
+      (effects (font (size 1.27 1.27)) hide)
+    )
+    (property "MPN" "0402B102K500NT" (at 181.61 134.62 0)
+      (effects (font (size 1.27 1.27)) hide)
+    )
+    (property "LCSC" "C1523" (at 181.61 134.62 0)
+      (effects (font (size 1.27 1.27)) hide)
+    )
+    (property "Type" "Basic" (at 181.61 134.62 0)
       (effects (font (size 1.27 1.27)) hide)
     )
@@
       (effects (font (size 1.524 1.524)) (justify left) hide)
     )
-    (property "Vendor" "Digikey" (at 128.27 71.12 0)
-      (effects (font (size 1.27 1.27)) hide)
-    )
-    (property "Vendor#" "296-48904-1-ND" (at 128.27 71.12 0)
+    (property "Vendor" "TI" (at 128.27 71.12 0)
+      (effects (font (size 1.27 1.27)) hide)
+    )
+    (property "Vendor#" "CSD88584Q5DC" (at 128.27 71.12 0)
       (effects (font (size 1.27 1.27)) hide)
     )
@@
     )
     (property "LCSC" "" (at 128.27 71.12 0)
+      (effects (font (size 1.27 1.27)) hide)
+    )
+    (property "Type" "Global" (at 128.27 71.12 0)
       (effects (font (size 1.27 1.27)) hide)
     )
@@
       (effects (font (size 1.27 1.27)) hide)
     )
+    (property "Type" "Extended" (at 128.27 118.11 0)
+      (effects (font (size 1.27 1.27)) hide)
+    )
     (pin "1")
     (pin "2")
@@
       (effects (font (size 1.27 1.27)) hide)
     )
+    (property "Type" "Extended" (at 97.79 62.23 0)
+      (effects (font (size 1.27 1.27)) hide)
+    )
     (pin "1")
     (pin "2")
@@
       (effects (font (size 1.27 1.27)) hide)
     )
-    (property "Vendor#" "C185450" (at 146.05 115.57 0)
-      (effects (font (size 1.27 1.27)) hide)
-    )
-    (property "MPN" "RC0402FR-071K78L " (at 146.05 115.57 0)
-      (effects (font (size 1.27 1.27)) hide)
-    )
-    (property "LCSC" "C185450" (at 146.05 115.57 0)
-      (effects (font (size 1.27 1.27)) hide)
-    )
+    (property "Vendor#" "C284379" (at 146.05 115.57 0)
+      (effects (font (size 1.27 1.27)) hide)
+    )
+    (property "MPN" "ARG02FTC1781" (at 146.05 115.57 0)
+      (effects (font (size 1.27 1.27)) hide)
+    )
+    (property "LCSC" "C284379" (at 146.05 115.57 0)
+      (effects (font (size 1.27 1.27)) hide)
+    )
+    (property "Type" "Extended" (at 146.05 115.57 0)
+      (effects (font (size 1.27 1.27)) hide)
+    )
