File: v3/O32controller.kicad_sch (KiCad schematic)
At the start: 44 parts, among them J1 BATT+, J13 PA15, J2 BATT+, J3 BATT-, J4 BATT-, J5 NTC, J6 SWD, J7 AuxUART, J8 RS485, J9 RS485, U1 STSPIN32F0ATR, U2 THVD1420DRLR, U3 MA732GQ-Z

Commit message: release v3.1 and generate gerbers
Parts:
- J13, J7: now left out of the parts list
Changed lines of the file:
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@@
   )
   (symbol (lib_id "Connector:Conn_01x01_Pin") (at 31.75 185.42 0) (unit 1)
-    (in_bom yes) (on_board yes) (dnp no) (fields_autoplaced)
+    (in_bom no) (on_board yes) (dnp no) (fields_autoplaced)
     (property "Reference" "J13" (at 32.385 180.34 0)
       (effects (font (size 1.27 1.27)))
@@
   )
   (symbol (lib_id "Connector:Conn_01x04_Pin") (at 31.75 170.18 0) (unit 1)
-    (in_bom yes) (on_board yes) (dnp no) (fields_autoplaced)
+    (in_bom no) (on_board yes) (dnp no) (fields_autoplaced)
     (property "Reference" "J7" (at 32.385 162.56 0)
       (effects (font (size 1.27 1.27)))
